File: circuits/cny70-board/cny70-board.kicad_sch (KiCad schematic)
At the start: 25 parts, among them J1 Out, Q1 2N3904, Q2 2N3904, Q3 2N3904, Q4 2N3904, U1 CNY70, U2 CNY70, U3 CNY70, U4 CNY70

Commit message: Line width changed
Path/spaces are now 0.3048/0.3048 mm (12/12 mil), and vias are 1.6-0.8 mm
Parts:
- Q1, Q2, Q3, Q4: footprint Package_TO_SOT_THT:TO-92_Inline -> Package_TO_SOT_THT:TO-92_Inline_Wide
Changed lines of the file:
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@@
       (effects (font (size 1.27 1.27)) (justify left))
     )
-    (property "Footprint" "Package_TO_SOT_THT:TO-92_Inline" (at 157.48 121.285 0)
+    (property "Footprint" "Package_TO_SOT_THT:TO-92_Inline_Wide" (at 157.48 121.285 0)
       (effects (font (size 1.27 1.27) italic) (justify left) hide)
     )
@@
       (effects (font (size 1.27 1.27)) (justify left))
     )
-    (property "Footprint" "Package_TO_SOT_THT:TO-92_Inline" (at 157.48 165.735 0)
+    (property "Footprint" "Package_TO_SOT_THT:TO-92_Inline_Wide" (at 157.48 165.735 0)
       (effects (font (size 1.27 1.27) italic) (justify left) hide)
     )
@@
       (effects (font (size 1.27 1.27)) (justify left))
     )
-    (property "Footprint" "Package_TO_SOT_THT:TO-92_Inline" (at 223.52 140.335 0)
+    (property "Footprint" "Package_TO_SOT_THT:TO-92_Inline_Wide" (at 223.52 140.335 0)
       (effects (font (size 1.27 1.27) italic) (justify left) hide)
     )
@@
       (effects (font (size 1.27 1.27)) (justify left))
     )
-    (property "Footprint" "Package_TO_SOT_THT:TO-92_Inline" (at 157.48 74.295 0)
+    (property "Footprint" "Package_TO_SOT_THT:TO-92_Inline_Wide" (at 157.48 74.295 0)
       (effects (font (size 1.27 1.27) italic) (justify left) hide)
     )
